File: radioboard.sch (EAGLE design)
At the start: 22 parts, among them Q1 8MHz, U1 STM32F302_303C2

Commit message: finished schematic, continued placing
Parts:
- removed LED2, LED3: (no value), misc:LEDCHIPLED_0805
- added C10, C12, C9: 10u, rcl:C-EUC0805
- added C11, C13: 100n, rcl:C-EUC0805
- added DWM1000: DWM1000, DWM1000:DWM1000
- added IC1: VREG-TS1117CW-3V3, we-power:VREG-TS1117CW-3V3
- added R5: 1k, rcl:R-US_M0805
- added R6: 47k, rcl:R-US_M0805
- added STAT1, STAT2: (no value), misc:LEDCHIPLED_0805
- R3: value 1k -> 47k
- U1: value STM32F302_303C2 -> STM32F302C8
- renumbered LED1 to STAT3
Connections:
- removed net N$15: U1A.PA9
- removed net N$9: LED3.A, R3.1
- new net DWM_IRQ: DWM1000.IRQ, U1A.PA15
- new net DWM_MISO: DWM1000.SPIMISO, U1A.PB4
- new net DWM_MOSI: DWM1000.SPIMOSI, U1A.PB5
- new net DWM_N_CS: DWM1000.SPICSN, U1A.PB6
- new net DWM_N_RST: DWM1000.RSTN, U1A.PB7
- new net DWM_SCK: DWM1000.SPICLK, U1A.PB3
- new net N$10: R5.2, STAT1.A
- new net N$5: R5.1, U1A.PC15-OSC_OUT
- net +3V3: now also C10.1, C11.1, C12.1, DWM1000.VDD1, DWM1000.VDD2, DWM1000.VDDA, IC1.VOUT
- net +5V: now also C9.1, IC1.VIN, R6.1
- net GND: now also C10.2, C11.2, C12.2, C13.2, C9.2, DWM1000.VSS1, DWM1000.VSS2, DWM1000.VSS3, DWM1000.VSS4, DWM1000.VSS5, IC1.GND, R3.2, STAT1.C, STAT2.C; no longer LED2.C, LED3.C
- net N$7: now also STAT2.A; no longer LED2.A
- net N$8: now also C13.1, R3.1, R6.2, U1A.PA3; no longer R3.2, U1A.PA15
Other:
- moved on the sheet: MOTSPI-1, MOTSPI-2, MOTSPI-3, MOTSPI-4, MOTSPI-5, MOTSPI-6, R2, R3, RPI-1, RPI-2, RPI-3, RPI-4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

Commit message: finished PCB
Parts:
- added ON: (no value), misc:LEDCHIPLED_0805
- added R7: 2.2k, rcl:R-US_M0805
- renumbered STAT1 to SYNC, STAT2 to RX/TX, STAT3 to BATT
Connections:
- new net N$9: ON.C, R7.2
- net +3V3: now also ON.A
- net GND: now also R7.1
